Commit message: puppy urdf prototype

File: robotdog_description/urdf/puppy.urdf (robot description, URDF)
Before this commit: robot puppy, 9 links, 8 joints
Links:
- added link LF_calf; visual cylinder length=0.08 radius=0.008
- added link LH_calf; visual cylinder length=0.08 radius=0.008
- added link RF_calf; visual cylinder length=0.08 radius=0.008
- added link RH_calf; visual cylinder length=0.08 radius=0.008
- link LF_hip: geometry visual cylinder length=0.0433 radius=0.015
- link LF_thigh: geometry visual cylinder length=0.064 radius=0.012
- link LH_hip: geometry visual cylinder length=0.0433 radius=0.015
- link LH_thigh: geometry visual cylinder length=0.064 radius=0.012
- link RF_hip: geometry visual cylinder length=0.0433 radius=0.015
- link RF_thigh: geometry visual cylinder length=0.064 radius=0.012
- link RH_hip: geometry visual cylinder length=0.0433 radius=0.015
- link RH_thigh: geometry visual cylinder length=0.064 radius=0.012
Joints:
- added joint LF_KFE: type revolute, parent LF_thigh, child LF_calf, origin xyz=0.0452 -0.0452 0 rpy=0 0 0, axis 0 0 1, limit lower=-0.785 upper=0.785 effort=1000.0 velocity=0.5
- added joint LH_KFE: type revolute, parent LH_thigh, child LH_calf, origin xyz=0.0452 -0.0452 0 rpy=0 0 0, axis 0 0 1, limit lower=-0.785 upper=0.785 effort=1000.0 velocity=0.5
- added joint RF_KFE: type revolute, parent RF_thigh, child RF_calf, origin xyz=-0.0452 -0.0452 0 rpy=0 0 0, axis 0 0 1, limit lower=-0.785 upper=0.785 effort=1000.0 velocity=0.5
- added joint RH_KFE: type revolute, parent RH_thigh, child RH_calf, origin xyz=-0.0452 -0.0452 0 rpy=0 0 0, axis 0 0 1, limit lower=-0.785 upper=0.785 effort=1000.0 velocity=0.5
- joint LF_HAA: limit lower=-1.74 upper=1.74 effort=1000.0 velocity=0.5 -> lower=-1.57 upper=1.57 effort=1000.0 velocity=0.5
- joint LF_HFE: limit lower=-1.74 upper=1.74 effort=1000.0 velocity=0.5 -> lower=-1.57 upper=1.57 effort=1000.0 velocity=0.5
- joint LH_HAA: limit lower=-1.74 upper=1.74 effort=1000.0 velocity=0.5 -> lower=-1.57 upper=1.57 effort=1000.0 velocity=0.5
- joint LH_HFE: limit lower=-1.74 upper=1.74 effort=1000.0 velocity=0.5 -> lower=-1.57 upper=1.57 effort=1000.0 velocity=0.5
- joint RF_HAA: limit lower=-1.74 upper=1.74 effort=1000.0 velocity=0.5 -> lower=-1.57 upper=1.57 effort=1000.0 velocity=0.5
- joint RF_HFE: limit lower=-1.74 upper=1.74 effort=1000.0 velocity=0.5 -> lower=-1.57 upper=1.57 effort=1000.0 velocity=0.5
- joint RH_HAA: limit lower=-1.74 upper=1.74 effort=1000.0 velocity=0.5 -> lower=-1.57 upper=1.57 effort=1000.0 velocity=0.5
- joint RH_HFE: limit lower=-1.74 upper=1.74 effort=1000.0 velocity=0.5 -> lower=-1.57 upper=1.57 effort=1000.0 velocity=0.5
